File: LED Ring PCB/LED Ring.kicad_pcb (KiCad board)
At the start: 2 copper layers, 22.9 x 22.9 mm, 8 parts

Commit message: Viewer and LED Ring Stuff
Parts:
- added DIN: TestPoint_Keystone_5015_Micro_Mini, TestPoint:TestPoint_Keystone_5015_Micro_Mini, B.Cu at (6.75, -7.00)
- added DOUT: TestPoint_Keystone_5015_Micro_Mini, TestPoint:TestPoint_Keystone_5015_Micro_Mini, B.Cu at (-6.75, -6.50)
- added GND: TestPoint_Keystone_5015_Micro_Mini, TestPoint:TestPoint_Keystone_5015_Micro_Mini, B.Cu at (8.50, 0.00)
- added VDD: TestPoint_Keystone_5015_Micro_Mini, TestPoint:TestPoint_Keystone_5015_Micro_Mini, B.Cu at (-6.25, 6.25)
- moved VDD 0.71 mm to (-6.50, 6.00), turned to -45 degrees
Routing:
- net Net-(J2-Pin_2): vias 0 -> 1
- net Net-(J1-Pin_2): vias 0 -> 1
